File: MorePCBDoodles.kicad_sch (KiCad schematic)
At the start: 102 parts, among them J1 USB_C_Receptacle, J2 Conn_01x04, J3 Conn_01x04, SW1 Push_Button, U1 RP2040, U2 AP2112K-3.3, U3 ww, U4 RP2040, U5 ww, U6 MAX7219, U7 ST25R3911B-AQF, X1 SMD3225-4, X2 SMD3225-4, Y1 Crystal_GND24

Commit message: Add files via upload
Parts:
- added C18: 1uF_50V, Capacitor_THT:CP_Radial_D4.0mm_P1.50mm, symbol PCM_SL_Capacitors:1uF_50V
- added C19, C20: 0.1uF, Capacitor_SMD:CP_Elec_3x5.3, symbol Device:C
- added D1: WS2812, LED_SMD:LED_WS2812_PLCC6_5.0x5.0mm_P1.6mm, symbol LED:WS2812
- added J4: RJ45_RB1-125B8G1A, Connector_RJ:RJ45_UDE_RB1-125B8G1A, symbol Connector:RJ45_RB1-125B8G1A
- added J5: JST_06, Connector_JST:JST_EH_B6B-EH-A_1x06_P2.50mm_Vertical, symbol PCM_SL_Connectors:JST_06
- added R4: 10k, Resistor_THT:R_Axial_DIN0207_L6.3mm_D2.5mm_P10.16mm_Horizontal, symbol PCM_SL_Resistors:10k
- added R5, R6, R7: 330ohm, Resistor_THT:R_Axial_DIN0207_L6.3mm_D2.5mm_P10.16mm_Horizontal, symbol PCM_SL_Resistors:330ohm
- added SW2, SW3, SW4: Push_Button, Button_Switch_SMD:SW_SPST_TS-1088-xR020, symbol PCM_SL_Devices:Push_Button
- added U8: W5500, Package_QFP:LQFP-48_7x7mm_P0.5mm, symbol Interface_Ethernet:W5500
- added Y2: 25MHz, Crystal:Crystal_SMD_3225-4Pin_3.2x2.5mm, symbol Device:Crystal
- C12, C13, C14, C15, C16: footprint (none) -> Capacitor_THT:CP_Axial_L10.0mm_D4.5mm_P15.00mm_Horizontal
- J1: footprint (none) -> Connector_USB:USB_C_Receptacle_Amphenol_124019772112A
- J2, J3: footprint (none) -> Connector_PinHeader_1.00mm:PinHeader_1x04_P1.00mm_Horizontal
- TP1, TP2: footprint (none) -> TestPoint:TestPoint_2Pads_Pitch2.54mm_Drill0.8mm
- U6: footprint (none) -> Package_SO:SOIC-24W_7.5x15.4mm_P1.27mm
- Y1: footprint (none) -> Crystal:Crystal_SMD_3225-4Pin_3.2x2.5mm
Connections:
- net at C1.1, C6.1, J2.2 (Pin_2)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: now also J5.1, R4.1, R5.1, R6.1, U8.11 (AVDD), U8.15 (AVDD), U8.17 (AVDD), U8.21 (AVDD), U8.28 (VDD), U8.4 (AVDD), U8.43 (PMODE2), U8.44 (PMODE1), U8.45 (PMODE0), U8.8 (AVDD)
- net at U4.11 (GPIO8): now also U8.36 (~{INT})
- net at U4.12 (GPIO9): now also U8.35 (MOSI)
- net at U4.13 (GPIO10): now also U8.34 (MISO)
- net at U4.14 (GPIO11): now also U8.33 (SCLK)
- net at U4.15 (GPIO12): now also U8.32 (~{SCS})
- net at C10.2, C12.2, C13.2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: now also C18.2, C19.2, D1.6 (VSS), J4.R10 (GND), J4.SH, J5.6, SW2.1, SW3.1, SW4.1, U8.14 (AGND), U8.16 (AGND), U8.19 (AGND), U8.29 (GND), U8.3 (AGND), U8.48 (AGND), U8.9 (AGND)
- net at U4.2 (GPIO0): now also J5.2
- net at U4.27 (GPIO16): no longer U7.31 (SCLK)
- net at U4.3 (GPIO1): now also J5.3
- net at U4.4 (GPIO2): now also J5.4
- net at U4.5 (GPIO3): now also J5.5
- net at U4.6 (GPIO4): now also SW4.2
- net at U4.7 (GPIO5): now also SW3.2
- net at U4.8 (GPIO6): now also SW2.2
- net at U4.9 (GPIO7): now also R7.1
- net at C11.2, C14.2, C16.2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: now also C15.1, C16.1, C17.2, TP2.1
- net at J1.A4 (VBUS), J1.A9 (VBUS), J1.B4 (VBUS)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: now also D1.3 (VCC), D1.5 (VDD)
- new net: J4.L3, R6.2
- new net: R4.2, U8.37 (~{RST})
- new net: J4.L2, R5.2
- new net: C19.1, U8.20 (TOCAP)
- new net: D1.2 (DIN), R7.2
- new net: J4.L1, U8.25 (LINKLED)
- new net: J4.L4, U8.27 (ACTLED)
- new net: J4.R1 (CT), U8.2 (TXP)
- new net: J4.R2 (TD1+), U8.1 (TXN)
- new net: J4.R3 (TD1-), U8.5 (RXN)
- new net: J4.R6 (TD3+), U8.6 (RXP)
- new net: U8.30 (XI/CLKIN), Y2.1
- new net: U8.31 (XO), Y2.2
- new net: C18.1, U8.22 (1V2O)
- no-connect marks 3 -> 10
